Commit message: update model with servo mesh

File: quaro_description/urdf/body.xacro (robot description, xacro)
@@ -1,36 +1,114 @@
 <?xml version="1.0"?>
 <robot name="quaro-body" xmlns:xacro="http://ros.org/wiki/xacro">
-  <xacro:property name="pi" value="3.1415"/>
-  <xacro:include filename="$(find quaro_description)/urdf/colors.xacro"/>
-  <xacro:include filename="$(find quaro_description)/urdf/leg.xacro"/>
-  <!-- first link -->
+  <!-- Sensor param will be used later when stereo camera and other sensors will be installed. -->
+  <xacro:macro name="body" params="sensors">
   <link name="front">
     <visual>
       <geometry>
-        <mesh filename="package://quaro_description/meshes/front.stl"/>
+        <mesh filename="package://quaro_description/meshes/front.stl" scale="${scale} ${scale} ${scale}"/>
       </geometry>
       <material name="pink"/>
-      <origin rpy="0 0 0" xyz="0 0 20"/>
+      <origin rpy="0 0 0" xyz="0 0 ${21*scale}"/>
     </visual>
+    <inertial>
+      <mass value="${60*gtoKg}" />
+      <inertia  ixx="${1*scale_mm2*gtoKg}"
+                ixy="${0*scale_mm2*gtoKg}"
+                ixz="${0*scale_mm2*gtoKg}"
+                iyy="${1*scale_mm2*gtoKg}"
+                iyz="${0*scale_mm2*gtoKg}"
+                izz="${1*scale_mm2*gtoKg}" />
+    </inertial>
+    <collision>
+       <geometry>
+         <mesh filename="package://quaro_description/meshes/front.stl" scale="${scale} ${scale} ${scale}"/>
+       </geometry>
+       <origin rpy="0 0 0" xyz="0 0 ${20*scale}"/>
+     </collision>
   </link>
   <link name="back">
     <visual>
       <geometry>
-        <mesh filename="package://quaro_description/meshes/back.stl"/>
+        <mesh filename="package://quaro_description/meshes/back.stl" scale="${scale} ${scale} ${scale}"/>
       </geometry>
       <material name="gray"/>
-      <origin rpy="0 0 0" xyz="-15 0 20"/>
+      <origin rpy="0 0 0" xyz="-${15*scale} 0 ${20*scale}"/>
+    </visual>
+    <inertial>
+      <mass value="${60*gtoKg}" />
+      <inertia  ixx="${1*scale_mm2*gtoKg}"
+                ixy="${0*scale_mm2*gtoKg}"
+                ixz="${0*scale_mm2*gtoKg}"
+                iyy="${1*scale_mm2*gtoKg}"
+                iyz="${0*scale_mm2*gtoKg}"
+                izz="${1*scale_mm2*gtoKg}" />
+    </inertial>
+    <collision>
+       <geometry>
+         <mesh filename="package://quaro_description/meshes/back.stl"/>
+       </geometry>
+       <origin rpy="0 0 0" xyz="-${15*scale} 0 ${20*scale}"/>
+     </collision>
+  </link>
+  <link name="chest-servo">
+    <visual>
+      <geometry>
+        <mesh filename="package://quaro_description/meshes/AX-12A.stl" scale="${scale} ${scale} ${scale}"/>
+      </geometry>
+      <material name="red"/>
+      <origin rpy="${pi/2} ${pi} 0" xyz="${0*scale} ${0*scale} ${0*scale}"/>
+    </visual>
+    <inertial>
+      <mass value="${600*gtoKg}" />
+      <inertia  ixx="${1*scale_mm2*gtoKg}"
+              ixy="${0*scale_mm2*gtoKg}"
+              ixz="${0*scale_mm2*gtoKg}"
+              iyy="${1*scale_mm2*gtoKg}"
+              iyz="${0*scale_mm2*gtoKg}"
+              izz="${1*scale_mm2*gtoKg}" />
+    </inertial>
+    <collision>
+       <geometry>
+         <mesh filename="package://quaro_description/meshes/AX-12A.stl" scale="${scale} ${scale} ${scale}"/>
+       </geometry>
+       <origin rpy="${pi/2} 0  ${pi/2}" xyz="-${15*scale} -${20*scale} -${20*scale}"/>
+     </collision>
+  </link>
+  <link name="spine">
+    <visual>
+      <geometry>
+        <mesh filename="package://quaro_description/meshes/link-chest.stl" scale="${scale} ${scale} ${scale}"/>
+      </geometry>
+      <material name="yellow"/>
+      <origin rpy="${pi/2} ${pi/2} 0" xyz="-${11*scale} ${22*scale} ${16*scale}"/>
     </visual>
   </link>
+  <joint name="servo-link" type="fixed">
+    <parent link="back"/>
+    <child link="chest-servo"/>
+    <origin rpy="0 0 0" xyz="-${5*scale} ${0*scale} ${0*scale}"/>
+  </joint>
   <joint name="chest" type="revolute">
-    <parent link="front"/>
-    <child link="back"/>
-    <origin rpy="0 0 0" xyz="-15 0 0"/>
+    <parent link="chest-servo"/>
+    <child link="spine"/>
+    <origin rpy="0 0 0" xyz="0 0 0"/>
     <axis xyz="0 1 0"/>
     <limit effort="1000.0" lower="${-pi/2}" upper="${pi/2}" velocity="0.5"/>
   </joint>
-  <xacro:leg n="0" x="150" y="90" angle="${1*pi/4}" parent="front"/>
-  <xacro:leg n="1" x="150" y="-90" angle="-${1*pi/4}" parent="front"/>
-  <xacro:leg n="2" x="-140" y="90" angle="${3*pi/4}" parent="back"/>
-  <xacro:leg n="3" x="-140" y="-90" angle="-${3*pi/4}" parent="back"/>
+  <joint name="last" type="fixed">
+    <parent link="spine"/>
+    <child link="front"/>
+    <origin ryp="0 0 0" xyz="${15 *scale} ${0*scale} ${0*scale}"/>
+  </joint>
+  <transmission name="chest">
+    <type>transmission_interface/SimpleTransmission</type>
+    <joint name="chest">
+      <hardwareInterface>hardware_interface/EffortJointInterface</hardwareInterface>
+    </joint>
+    <actuator name="motor-chest">
+      <hardwareInterface>hardware_interface/EffortJointInterface</hardwareInterface>
+      <mechanicalReduction>1</mechanicalReduction>
+    </actuator>
+  </transmission>
+  </xacro:macro>
 </robot>

File: quaro_description/urdf/leg.xacro (robot description, xacro)
@@ -3,53 +3,140 @@
   <!-- parameter n is the leg number-->
   <xacro:macro name="leg" params="n x y angle parent">
-  <!-- first link -->
-  <link name="thigh${n}">
-    <visual>
-      <geometry>
-        <mesh filename="package://quaro_description/meshes/thigh.stl"/>
-      </geometry>
-      <material name="red"/>
-      <origin rpy="${pi/2} 0  ${pi/2}" xyz="-15 -20 -20"/>
-    </visual>
-  </link>
-  <link name="shin${n}">
-    <visual>
-      <geometry>
-        <mesh filename="package://quaro_description/meshes/shin.stl"/>
-      </geometry>
-      <material name="blue"/>
-      <origin rpy="0 0 0" xyz="20 -20 -20"/>
-    </visual>
-  </link>
-  <joint name="knee${n}" type="revolute">
-    <parent link="thigh${n}"/>
-    <child link="shin${n}"/>
-    <origin rpy="${pi/2} 0 0" xyz="30 0 0"/>
-    <axis xyz="0 0 1"/>
-    <limit effort="1000.0" lower="${-pi/2}" upper="${pi/2}" velocity="0.5"/>
-  </joint>
-  <link name="foot${n}">
-    <visual>
-      <geometry>
-        <mesh filename="package://quaro_description/meshes/foot.stl"/>
-      </geometry>
-      <material name="green"/>
-      <origin ryp="0 0 0" xyz="20 -105 -20"/>
-    </visual>
-  </link>
-  <joint name="ankle${n}" type="revolute">
-    <parent link="shin${n}"/>
-    <child link="foot${n}"/>
-    <origin rpy="0 0 0" xyz="70 0 0"/>
-    <axis xyz="0 0 1"/>
-    <limit effort="1000.0" lower="${-pi/2}" upper="${pi/2}" velocity="0.5"/>
-  </joint>
-  <joint name="hip${n}" type="revolute">
-    <parent link="${parent}"/>
-    <child link="thigh${n}"/>
-    <origin rpy="0 0 ${angle}" xyz="${x} ${y} -10"/>
-    <axis xyz="0 0 1"/>
-    <limit effort="1000.0" lower="-${pi/2}" upper="${pi/2}" velocity="0.5"/>
-  </joint>
-</xacro:macro>
+    <!-- first link -->
+    <link name="hip${n}-servo">
+      <visual>
+        <geometry>
+          <mesh filename="package://quaro_description/meshes/AX-12A.stl" scale="${scale} ${scale} ${scale}"/>
+        </geometry>
+        <material name="red"/>
+        <origin rpy="0 ${pi} 0" xyz="${0*scale} ${0*scale} ${0*scale}"/>
+      </visual>
+      <inertial>
+        <mass value="${600*gtoKg}" />
+        <inertia  ixx="${1*scale_mm2*gtoKg}"
+                ixy="${0*scale_mm2*gtoKg}"
+                ixz="${0*scale_mm2*gtoKg}"
+                iyy="${1*scale_mm2*gtoKg}"
+                iyz="${0*scale_mm2*gtoKg}"
+                izz="${1*scale_mm2*gtoKg}" />
+      </inertial>
+      <collision>
+         <geometry>
+           <mesh filename="package://quaro_description/meshes/AX-12A.stl" scale="${scale} ${scale} ${scale}"/>
+         </geometry>
+         <origin rpy="${pi/2} 0  ${pi/2}" xyz="-${15*scale} -${20*scale} -${20*scale}"/>
+       </collision>
+    </link>
+    <joint name="hip-link${n}" type="fixed">
+      <parent link="${parent}"/>
+      <child link="hip${n}-servo"/>
+      <origin rpy="0 0 ${angle}" xyz="${x*scale} ${y*scale} ${0*scale}"/>
+    </joint>
+    <link name="thigh${n}">
+      <visual>
+        <geometry>
+          <mesh filename="package://quaro_description/meshes/link-hip.stl" scale="${scale} ${scale} ${scale}"/>
+        </geometry>
+        <material name="red"/>
+        <origin rpy="${pi} 0 ${pi/2}" xyz="-${11.04*scale} -${11.05*scale} ${23.97*scale}"/>
+      </visual>
+    </link>
+    <joint name="hip${n}" type="revolute">
+      <parent link="hip${n}-servo"/>
+      <child link="thigh${n}"/>
+      <origin rpy="0 0 0" xyz="${0*scale} 0 0"/>
+      <axis xyz="0 0 1"/>
+      <limit effort="1000.0" lower="${-pi/3}" upper="${pi/3}" velocity="0.5"/>
+    </joint>
+    <link name="knee${n}-servo">
+      <visual>
+        <geometry>
+          <mesh filename="package://quaro_description/meshes/AX-12A.stl" scale="${scale} ${scale} ${scale}"/>
+        </geometry>
+        <material name="blue"/>
+        <origin rpy="0 0 0" xyz="${0*scale} ${0*scale} ${0*scale}"/>
+      </visual>
+      <inertial>
+        <mass value="${600*gtoKg}" />
+        <inertia  ixx="${1*scale_mm2*gtoKg}"
+                ixy="${0*scale_mm2*gtoKg}"
+                ixz="${0*scale_mm2*gtoKg}"
+                iyy="${1*scale_mm2*gtoKg}"
+                iyz="${0*scale_mm2*gtoKg}"
+                izz="${1*scale_mm2*gtoKg}" />
+      </inertial>
+      <collision>
+         <geometry>
+           <mesh filename="package://quaro_description/meshes/AX-12A.stl" scale="${scale} ${scale} ${scale}"/>
+         </geometry>
+         <origin rpy="0 0 0" xyz="${0*scale} ${0*scale} ${0*scale}"/>
+       </collision>
+    </link>
+    <joint name="knee${n}-link" type="fixed">
+      <parent link="thigh${n}"/>
+      <child link="knee${n}-servo"/>
+      <origin rpy="-${pi/2} ${pi} 0" xyz="${59.35*scale} ${0*scale} 0"/>
+    </joint>
+    <link name="shin${n}">
+      <visual>
+        <geometry>
+          <mesh filename="package://quaro_description/meshes/link-knee.stl" scale="${scale} ${scale} ${scale}"/>
+        </geometry>
+        <material name="blue"/>
+        <origin rpy="${pi} ${pi} -${pi/2}" xyz="${11.04*scale} -${18.05*scale} -${23.97*scale}"/>
+      </visual>
+    </link>
+    <joint name="knee${n}" type="revolute">
+      <parent link="knee${n}-servo"/>
+      <child link="shin${n}"/>
+      <origin rpy="0 0 0" xyz="${0*scale} 0 0"/>
+      <axis xyz="0 0 1"/>
+      <limit effort="1000.0" lower="${-pi/3}" upper="${pi/3}" velocity="0.5"/>
+    </joint>
+    <link name="ankle${n}-servo">
+      <visual>
+        <geometry>
+          <mesh filename="package://quaro_description/meshes/AX-12A.stl" scale="${scale} ${scale} ${scale}"/>
+        </geometry>
+        <material name="green"/>
+        <origin ryp="0 0 0" xyz="${0*scale} -${0*scale} -${0*scale}"/>
+      </visual>
+      <inertial>
+        <mass value="${600*gtoKg}" />
+        <inertia  ixx="${1*scale_mm2*gtoKg}"
+                ixy="${0*scale_mm2*gtoKg}"
+                ixz="${0*scale_mm2*gtoKg}"
+                iyy="${1*scale_mm2*gtoKg}"
+                iyz="${0*scale_mm2*gtoKg}"
+                izz="${1*scale_mm2*gtoKg}" />
+      </inertial>
+      <collision>
+         <geometry>
+           <mesh filename="package://quaro_description/meshes/AX-12A.stl" scale="${scale} ${scale} ${scale}"/>
+         </geometry>
+         <origin rpy="0 0 0" xyz="${0*scale} -${0*scale} -${0*scale}"/>
+       </collision>
+    </link>
+    <joint name="ankle${n}-link" type="fixed">
+      <parent link="shin${n}"/>
+      <child link="ankle${n}-servo"/>
+      <origin rpy="0 0 0" xyz="-${59.41*scale} 0 0"/>
+    </joint>
+    <link name="foot${n}">
+      <visual>
+        <geometry>
+          <mesh filename="package://quaro_description/meshes/link-foot.stl" scale="${scale} ${scale} ${scale}"/>
+        </geometry>
+        <material name="green"/>
+        <origin ryp="0 0 0" xyz="${0*scale} -${0*scale} -${22*scale}"/>
+      </visual>
+    </link>
+    <joint name="ankle${n}" type="revolute">
+      <parent link="ankle${n}-servo"/>
+      <child link="foot${n}"/>
+      <origin rpy="0 ${pi} 0" xyz="${0*scale} 0 0"/>
+      <axis xyz="0 0 1"/>
+      <limit effort="1000.0" lower="${-pi/3}" upper="${pi/3}" velocity="0.5"/>
+    </joint>
+  </xacro:macro>
 </robot>
