Commit message: renamed files and created new directories

File: quaro_description/urdf/quaro.gazebo.xacro (robot description, xacro)
@@ -48,7 +48,20 @@
   </xacro:macro>
   <xacro:macro name="leg_gazebo" params="n">
+    <xacro:red name="hip${n}-servo"/>
     <xacro:red name="thigh${n}"/>
+    <xacro:red name="knee{n}-servo"/>
     <xacro:blue name="shin${n}"/>
+    <xacro:green name="ankle${n}-servo"/>
     <xacro:green name="foot${n}"/>
+    <transmission name="hip${n}">
+      <type>transmission_interface/SimpleTransmission</type>
+      <joint name="hip${n}">
+        <hardwareInterface>hardware_interface/EffortJointInterface</hardwareInterface>
+      </joint>
+      <actuator name="motor-hip${n}">
+        <hardwareInterface>hardware_interface/EffortJointInterface</hardwareInterface>
+        <mechanicalReduction>1</mechanicalReduction>
+      </actuator>
+    </transmission>
     <transmission name="knee${n}">
       <type>transmission_interface/SimpleTransmission</type>
@@ -71,14 +84,4 @@
       </actuator>
     </transmission>
-    <transmission name="hip${n}">
-      <type>transmission_interface/SimpleTransmission</type>
-      <joint name="hip${n}">
-        <hardwareInterface>hardware_interface/EffortJointInterface</hardwareInterface>
-      </joint>
-      <actuator name="motor-hip${n}">
-        <hardwareInterface>hardware_interface/EffortJointInterface</hardwareInterface>
-        <mechanicalReduction>1</mechanicalReduction>
-      </actuator>
-    </transmission>
   </xacro:macro>
   <!-- Base -->

File: quaro_description/urdf/quaro.xacro (robot description, xacro)
@@ -2,8 +2,9 @@
 <robot name="quaro-body" xmlns:xacro="http://ros.org/wiki/xacro">
   <xacro:property name="pi" value="3.1415"/>
-  <xacro:include filename="$(find quaro_description)/urdf/colors.xacro"/>
-  <xacro:include filename="$(find quaro_description)/urdf/leg.xacro"/>
-  <xacro:include filename="$(find quaro_description)/urdf/body.xacro"/>
-  <xacro:include filename="$(find quaro_description)/urdf/robot.gazebo"/>
+  <xacro:property name="version" value=".0.0"/>
+  <xacro:include filename="$(find quaro_description)/urdf/common/colors.xacro"/>
+  <xacro:include filename="$(find quaro_description)/urdf/leg/leg${version}.xacro"/>
+  <xacro:include filename="$(find quaro_description)/urdf/body/body${version}.xacro"/>
+  <xacro:include filename="$(find quaro_description)/urdf/quaro.gazebo.xacro"/>
   <xacro:property name="scale" value="${0.01}"/>
   <xacro:property name="scale_mm" value="${1e-3*scale}"/>
