Commit message: last stage of the work

File: quaro_description/urdf/leg/leg.0.0.xacro (robot description, xacro)
@@ -132,4 +132,10 @@
       <limit effort="${effort}" lower="${-pi/3}" upper="${pi/3}" velocity="${velocity}"/>
     </joint>
+    <link name="eff${n}"/>
+    <joint name="eff${n}-joint" type="fixed">
+      <parent link="foot${n}"/>
+      <child link="eff${n}"/>
+      <origin xyz="${70*scale} -${115*scale} 0" rpy="-${pi/2} 0 0"/>
+    </joint>
   </xacro:macro>
 </robot>

File: quaro_description/urdf/quaro.xacro (robot description, xacro)
@@ -22,7 +22,11 @@
   </joint>
   <xacro:body sensors="none"/>
+  <!-- Front Left -->
   <xacro:leg n="0" x="132.63" y="74.77" z="-21" rpy="0 0 ${1*pi/4}" parent="front"/>
+  <!-- Front Right -->
   <xacro:leg n="1" x="132.63" y="-74.77" z="-21" rpy="0 0 -${1*pi/4}" parent="front"/>
+  <!-- Back Left -->
   <xacro:leg n="2" x="-107.63" y="74.77" z="-21" rpy="0 0 ${3*pi/4}" parent="back"/>
+  <!-- Back Right -->
   <xacro:leg n="3" x="-107.63" y="-74.77" z="-21" rpy="0 0 -${3*pi/4}" parent="back"/>
 </robot>
