Commit message: updtate the meshes to get an origin placed on the COM and adapted the urdf file

File: quaro_description/urdf/body/body.0.0.xacro (robot description, xacro)
@@ -3,4 +3,79 @@
   <!-- Sensor param will be used later when stereo camera and other sensors will be installed. -->
   <xacro:macro name="body" params="sensors">
+  <link name="back">
+    <visual>
+      <geometry>
+        <mesh filename="package://quaro_description/meshes/back.stl" scale="${scale} ${scale} ${scale}"/>
+      </geometry>
+      <material name="gray"/>
+      <origin rpy="0 0 0" xyz="${0*scale} 0 ${0*scale}"/>
+    </visual>
+    <inertial>
+      <mass value="${60*gtoKg}" />
+      <origin rpy="0 0 0" xyz="-${54.98*scale} ${0*scale} -${21.33*scale}"/>
+      <inertia  ixx="${1*scale_mm2*gtoKg}"
+                ixy="${0*scale_mm2*gtoKg}"
+                ixz="${0*scale_mm2*gtoKg}"
+                iyy="${1*scale_mm2*gtoKg}"
+                iyz="${0*scale_mm2*gtoKg}"
+                izz="${1*scale_mm2*gtoKg}" />
+    </inertial>
+    <collision>
+       <geometry>
+         <mesh filename="package://quaro_description/meshes/back.stl" scale="${scale} ${scale} ${scale}"/>
+       </geometry>
+       <origin rpy="0 0 0" xyz="${0*scale} 0 ${0*scale}"/>
+    </collision>
+  </link>
+  <link name="chest-servo">
+    <visual>
+      <geometry>
+        <mesh filename="package://quaro_description/meshes/AX-12A.stl" scale="${scale} ${scale} ${scale}"/>
+      </geometry>
+      <material name="red"/>
+      <origin rpy="0 0 0" xyz="${0*scale} ${0*scale} ${0*scale}"/>
+    </visual>
+    <inertial>
+      <mass value="${60*gtoKg}" />
+      <origin rpy="0 0 0" xyz="${12.61*scale} ${0*scale} ${1.21*scale}"/>
+      <inertia  ixx="${1*scale_mm2*gtoKg}"
+              ixy="${0*scale_mm2*gtoKg}"
+              ixz="${0*scale_mm2*gtoKg}"
+              iyy="${1*scale_mm2*gtoKg}"
+              iyz="${0*scale_mm2*gtoKg}"
+              izz="${1*scale_mm2*gtoKg}" />
+    </inertial>
+    <collision>
+       <geometry>
+         <mesh filename="package://quaro_description/meshes/AX-12A.stl" scale="${scale} ${scale} ${scale}"/>
+       </geometry>
+       <origin rpy="0 0 0" xyz="${0*scale} ${0*scale} ${0*scale}"/>
+     </collision>
+  </link>
+  <link name="spine">
+    <visual>
+      <geometry>
+        <mesh filename="package://quaro_description/meshes/link-chest.stl" scale="${scale} ${scale} ${scale}"/>
+      </geometry>
+      <material name="yellow"/>
+      <origin rpy="0 0 0" xyz="${16.58*scale} -${0.56*scale} ${0*scale}"/>
+    </visual>
+    <inertial>
+      <mass value="${60*gtoKg}" />
+      <origin rpy="0 0 0" xyz="${0*scale} -${0.56*scale} ${0*scale}"/>
+      <inertia  ixx="${1*scale_mm2*gtoKg}"
+                ixy="${0*scale_mm2*gtoKg}"
+                ixz="${0*scale_mm2*gtoKg}"
+                iyy="${1*scale_mm2*gtoKg}"
+                iyz="${0*scale_mm2*gtoKg}"
+                izz="${1*scale_mm2*gtoKg}" />
+    </inertial>
+    <collision>
+       <geometry>
+         <mesh filename="package://quaro_description/meshes/link-chest.stl" scale="${scale} ${scale} ${scale}"/>
+       </geometry>
+       <origin rpy="0 0 0" xyz="${16.58*scale} -${0.56*scale} ${0*scale}"/>
+     </collision>
+  </link>
   <link name="front">
     <visual>
@@ -9,8 +84,9 @@
       </geometry>
       <material name="pink"/>
-      <origin rpy="0 0 0" xyz="0 0 ${21*scale}"/>
+      <origin rpy="${0} ${0} ${0}" xyz="${0*scale} ${0*scale} ${0*scale}"/>
     </visual>
     <inertial>
       <mass value="${60*gtoKg}" />
+      <origin rpy="0 0 0" xyz="${71.80*scale} ${0*scale} -${24.62*scale}"/>
       <inertia  ixx="${1*scale_mm2*gtoKg}"
                 ixy="${0*scale_mm2*gtoKg}"
@@ -24,73 +100,16 @@
          <mesh filename="package://quaro_description/meshes/front.stl" scale="${scale} ${scale} ${scale}"/>
        </geometry>
-       <origin rpy="0 0 0" xyz="0 0 ${20*scale}"/>
+       <origin rpy="0 0 0" xyz="0 0 ${0*scale}"/>
      </collision>
-  </link>
-  <link name="back">
-    <visual>
-      <geometry>
-        <mesh filename="package://quaro_description/meshes/back.stl" scale="${scale} ${scale} ${scale}"/>
-      </geometry>
-      <material name="gray"/>
-      <origin rpy="0 0 0" xyz="-${15*scale} 0 ${20*scale}"/>
-    </visual>
-    <inertial>
-      <mass value="${60*gtoKg}" />
-      <inertia  ixx="${1*scale_mm2*gtoKg}"
-                ixy="${0*scale_mm2*gtoKg}"
-                ixz="${0*scale_mm2*gtoKg}"
-                iyy="${1*scale_mm2*gtoKg}"
-                iyz="${0*scale_mm2*gtoKg}"
-                izz="${1*scale_mm2*gtoKg}" />
-    </inertial>
-    <collision>
-       <geometry>
-         <mesh filename="package://quaro_description/meshes/back.stl"/>
-       </geometry>
-       <origin rpy="0 0 0" xyz="-${15*scale} 0 ${20*scale}"/>
-     </collision>
-  </link>
-  <link name="chest-servo">
-    <visual>
-      <geometry>
-        <mesh filename="package://quaro_description/meshes/AX-12A.stl" scale="${scale} ${scale} ${scale}"/>
-      </geometry>
-      <material name="red"/>
-      <origin rpy="${pi/2} ${pi} 0" xyz="${0*scale} ${0*scale} ${0*scale}"/>
-    </visual>
-    <inertial>
-      <mass value="${600*gtoKg}" />
-      <inertia  ixx="${1*scale_mm2*gtoKg}"
-              ixy="${0*scale_mm2*gtoKg}"
-              ixz="${0*scale_mm2*gtoKg}"
-              iyy="${1*scale_mm2*gtoKg}"
-              iyz="${0*scale_mm2*gtoKg}"
-              izz="${1*scale_mm2*gtoKg}" />
-    </inertial>
-    <collision>
-       <geometry>
-         <mesh filename="package://quaro_description/meshes/AX-12A.stl" scale="${scale} ${scale} ${scale}"/>
-       </geometry>
-       <origin rpy="${pi/2} 0  ${pi/2}" xyz="-${15*scale} -${20*scale} -${20*scale}"/>
-     </collision>
-  </link>
-  <link name="spine">
-    <visual>
-      <geometry>
-        <mesh filename="package://quaro_description/meshes/link-chest.stl" scale="${scale} ${scale} ${scale}"/>
-      </geometry>
-      <material name="yellow"/>
-      <origin rpy="${pi/2} ${pi/2} 0" xyz="-${11*scale} ${22*scale} ${16*scale}"/>
-    </visual>
   </link>
   <joint name="servo-link" type="fixed">
     <parent link="back"/>
     <child link="chest-servo"/>
-    <origin rpy="0 0 0" xyz="-${5*scale} ${0*scale} ${0*scale}"/>
+    <origin rpy="${pi/2} ${pi} 0" xyz="${0*scale} -${0.17*scale} -${21*scale}"/>
   </joint>
   <joint name="chest" type="revolute">
     <parent link="chest-servo"/>
     <child link="spine"/>
-    <origin rpy="0 0 0" xyz="0 0 0"/>
+    <origin rpy="${-pi/2} ${0} ${-pi}" xyz="-${0*scale} -${0*scale} ${0*scale}"/>
     <axis xyz="0 1 0"/>
     <limit effort="1000.0" lower="${-pi/2}" upper="${pi/2}" velocity="0.5"/>
@@ -99,16 +118,6 @@
     <parent link="spine"/>
     <child link="front"/>
-    <origin ryp="0 0 0" xyz="${15 *scale} ${0*scale} ${0*scale}"/>
+    <origin ryp="${0} ${0} ${0}" xyz="${16.58*scale} ${0*scale} ${21*scale}"/>
   </joint>
-  <transmission name="chest">
-    <type>transmission_interface/SimpleTransmission</type>
-    <joint name="chest">
-      <hardwareInterface>hardware_interface/EffortJointInterface</hardwareInterface>
-    </joint>
-    <actuator name="motor-chest">
-      <hardwareInterface>hardware_interface/EffortJointInterface</hardwareInterface>
-      <mechanicalReduction>1</mechanicalReduction>
-    </actuator>
-  </transmission>
   </xacro:macro>
 </robot>

File: quaro_description/urdf/leg/leg.0.0.xacro (robot description, xacro)
@@ -2,5 +2,5 @@
 <robot name="quaro-leg" xmlns:xacro="http://ros.org/wiki/xacro">
   <!-- parameter n is the leg number-->
-  <xacro:macro name="leg" params="n x y angle parent">
+  <xacro:macro name="leg" params="n x y z rpy parent">
     <!-- first link -->
     <link name="hip${n}-servo">
@@ -13,5 +13,6 @@
       </visual>
       <inertial>
-        <mass value="${600*gtoKg}" />
+        <mass value="${60*gtoKg}" />
+        <origin rpy="0 0 0" xyz="${12.61*scale} ${0*scale} ${1.21*scale}"/>
         <inertia  ixx="${1*scale_mm2*gtoKg}"
                 ixy="${0*scale_mm2*gtoKg}"
@@ -25,5 +26,5 @@
            <mesh filename="package://quaro_description/meshes/AX-12A.stl" scale="${scale} ${scale} ${scale}"/>
          </geometry>
-         <origin rpy="${pi/2} 0  ${pi/2}" xyz="-${15*scale} -${20*scale} -${20*scale}"/>
+         <origin rpy="0 ${pi} 0" xyz="${0*scale} ${0*scale} ${0*scale}"/>
        </collision>
     </link>
@@ -31,5 +32,5 @@
       <parent link="${parent}"/>
       <child link="hip${n}-servo"/>
-      <origin rpy="0 0 ${angle}" xyz="${x*scale} ${y*scale} ${0*scale}"/>
+      <origin rpy="${rpy}" xyz="${x*scale} ${y*scale} ${z*scale}"/>
     </joint>
     <link name="thigh${n}">
@@ -39,11 +40,27 @@
         </geometry>
         <material name="red"/>
-        <origin rpy="${pi} 0 ${pi/2}" xyz="-${11.04*scale} -${11.05*scale} ${23.97*scale}"/>
+        <origin rpy="${0} 0 -${pi/2}" xyz="${24.10*scale} -${0*scale} -${0*scale}"/>
       </visual>
+      <inertial>
+        <mass value="${60*gtoKg}" />
+        <origin rpy="${pi} 0 ${pi/2}" xyz="${24.10*scale} -${0*scale} -${0*scale}"/>
+        <inertia  ixx="${1*scale_mm2*gtoKg}"
+                ixy="${0*scale_mm2*gtoKg}"
+                ixz="${0*scale_mm2*gtoKg}"
+                iyy="${1*scale_mm2*gtoKg}"
+                iyz="${0*scale_mm2*gtoKg}"
+                izz="${1*scale_mm2*gtoKg}" />
+      </inertial>
+      <collision>
+         <geometry>
+           <mesh filename="package://quaro_description/meshes/link-hip.stl" scale="${scale} ${scale} ${scale}"/>
+         </geometry>
+         <origin rpy="${0} 0 -${pi/2}" xyz="${24.10*scale} -${0*scale} -${0*scale}"/>
+       </collision>
     </link>
     <joint name="hip${n}" type="revolute">
       <parent link="hip${n}-servo"/>
       <child link="thigh${n}"/>
-      <origin rpy="0 0 0" xyz="${0*scale} 0 0"/>
+      <origin rpy="0 0 0" xyz="${0*scale} ${0*scale} ${0*scale}"/>
       <axis xyz="0 0 1"/>
       <limit effort="1000.0" lower="${-pi/3}" upper="${pi/3}" velocity="0.5"/>
@@ -55,8 +72,9 @@
         </geometry>
         <material name="blue"/>
-        <origin rpy="0 0 0" xyz="${0*scale} ${0*scale} ${0*scale}"/>
+        <origin rpy="${0} 0 ${0}" xyz="-${0*scale} -${0*scale} ${0*scale}"/>
       </visual>
       <inertial>
-        <mass value="${600*gtoKg}" />
+        <mass value="${60*gtoKg}" />
+        <origin rpy="0 0 0" xyz="${12.61*scale} ${0*scale} ${1.21*scale}"/>
         <inertia  ixx="${1*scale_mm2*gtoKg}"
                 ixy="${0*scale_mm2*gtoKg}"
@@ -76,5 +94,5 @@
       <parent link="thigh${n}"/>
       <child link="knee${n}-servo"/>
-      <origin rpy="-${pi/2} ${pi} 0" xyz="${59.35*scale} ${0*scale} 0"/>
+      <origin rpy="-${pi/2} ${pi} 0" xyz="${57.35*scale} ${0.07*scale} -${0.5*scale}"/>
     </joint>
     <link name="shin${n}">
@@ -84,6 +102,22 @@
         </geometry>
         <material name="blue"/>
-        <origin rpy="${pi} ${pi} -${pi/2}" xyz="${11.04*scale} -${18.05*scale} -${23.97*scale}"/>
+        <origin rpy="${0} ${pi/2} ${pi/2}" xyz="-${23.63*scale} ${0*scale} ${0.31*scale}"/>
       </visual>
+      <inertial>
+        <mass value="${60*gtoKg}" />
+        <origin rpy="${0} ${pi/2} ${pi/2}" xyz="-${23.63*scale} ${0*scale} ${0.31*scale}"/>
+        <inertia  ixx="${1*scale_mm2*gtoKg}"
+                ixy="${0*scale_mm2*gtoKg}"
+                ixz="${0*scale_mm2*gtoKg}"
+                iyy="${1*scale_mm2*gtoKg}"
+                iyz="${0*scale_mm2*gtoKg}"
+                izz="${1*scale_mm2*gtoKg}" />
+      </inertial>
+      <collision>
+         <geometry>
+           <mesh filename="package://quaro_description/meshes/link-knee.stl" scale="${scale} ${scale} ${scale}"/>
+         </geometry>
+         <origin rpy="${0} ${pi/2} ${pi/2}" xyz="-${23.63*scale} ${0*scale} ${0.31*scale}"/>
+       </collision>
     </link>
     <joint name="knee${n}" type="revolute">
@@ -100,8 +134,8 @@
         </geometry>
         <material name="green"/>
-        <origin ryp="0 0 0" xyz="${0*scale} -${0*scale} -${0*scale}"/>
+        <origin rpy="${0} 0 ${0}" xyz="-${0*scale} -${0*scale} ${0*scale}"/>
       </visual>
       <inertial>
-        <mass value="${600*gtoKg}" />
+        <mass value="${60*gtoKg}" />
         <inertia  ixx="${1*scale_mm2*gtoKg}"
                 ixy="${0*scale_mm2*gtoKg}"
@@ -111,4 +145,5 @@
                 izz="${1*scale_mm2*gtoKg}" />
       </inertial>
+      <origin rpy="0 0 0" xyz="${12.61*scale} ${0*scale} ${1.21*scale}"/>
       <collision>
          <geometry>
@@ -121,5 +156,5 @@
       <parent link="shin${n}"/>
       <child link="ankle${n}-servo"/>
-      <origin rpy="0 0 0" xyz="-${59.41*scale} 0 0"/>
+      <origin rpy="${0} ${0} ${0}" xyz="-${58*scale} 0 0"/>
     </joint>
     <link name="foot${n}">
@@ -129,6 +164,22 @@
         </geometry>
         <material name="green"/>
-        <origin ryp="0 0 0" xyz="${0*scale} -${0*scale} -${22*scale}"/>
+        <origin rpy="${0} 0 ${0}" xyz="${35.02*scale} -${28.64*scale} ${2.64*scale}"/>
       </visual>
+      <inertial>
+        <mass value="${60*gtoKg}" />
+        <origin ryp="0 0 0" xyz="${35.02*scale} -${28.64*scale} ${2.64*scale}"/>
+        <inertia  ixx="${1*scale_mm2*gtoKg}"
+                ixy="${0*scale_mm2*gtoKg}"
+                ixz="${0*scale_mm2*gtoKg}"
+                iyy="${1*scale_mm2*gtoKg}"
+                iyz="${0*scale_mm2*gtoKg}"
+                izz="${1*scale_mm2*gtoKg}" />
+      </inertial>
+      <collision>
+         <geometry>
+           <mesh filename="package://quaro_description/meshes/link-foot.stl" scale="${scale} ${scale} ${scale}"/>
+         </geometry>
+           <origin rpy="${0} 0 ${0}" xyz="${35.02*scale} -${28.64*scale} ${2.64*scale}"/>
+       </collision>
     </link>
     <joint name="ankle${n}" type="revolute">

File: quaro_description/urdf/quaro.gazebo.xacro (robot description, xacro)
@@ -50,5 +50,5 @@
     <xacro:red name="hip${n}-servo"/>
     <xacro:red name="thigh${n}"/>
-    <xacro:red name="knee{n}-servo"/>
+    <xacro:blue name="knee${n}-servo"/>
     <xacro:blue name="shin${n}"/>
     <xacro:green name="ankle${n}-servo"/>
@@ -85,7 +85,19 @@
     </transmission>
   </xacro:macro>
+  <transmission name="chest">
+    <type>transmission_interface/SimpleTransmission</type>
+    <joint name="chest">
+      <hardwareInterface>hardware_interface/EffortJointInterface</hardwareInterface>
+    </joint>
+    <actuator name="motor-chest">
+      <hardwareInterface>hardware_interface/EffortJointInterface</hardwareInterface>
+      <mechanicalReduction>1</mechanicalReduction>
+    </actuator>
+  </transmission>
   <!-- Base -->
+  <xacro:grey name="back"/>
+  <xacro:yellow name="chest-servo"/>
+  <xacro:yellow name="spine"/>
   <xacro:black name="front"/>
-  <xacro:grey name="back"/>
   <xacro:leg_gazebo n="0"/>
   <xacro:leg_gazebo n="1"/>

File: quaro_description/urdf/quaro.xacro (robot description, xacro)
@@ -13,4 +13,16 @@
   <xacro:property name="angle_lim_low" value="${-8/18*pi}"/>
   <xacro:property name="angle_lim_high" value="${8/18*pi}"/>
+  <!-- first link -->
+  <link name="dummy-link"/>
+  <joint name="dummy-base" type="fixed">
+    <parent link="dummy-link"/>
+    <child link="back"/>
+    <origin rpy="0 0 0" xyz="${0*scale} ${0*scale} ${200*scale}"/>
+  </joint>
+  <xacro:body sensors="none"/>
+  <xacro:leg n="0" x="132.63" y="74.77" z="-21" rpy="0 0 ${1*pi/4}" parent="front"/>
+  <xacro:leg n="1" x="132.63" y="-74.77" z="-21" rpy="0 0 -${1*pi/4}" parent="front"/>
+  <xacro:leg n="2" x="-107.63" y="74.77" z="-21" rpy="0 0 ${3*pi/4}" parent="back"/>
+  <xacro:leg n="3" x="-107.63" y="-74.77" z="-21" rpy="0 0 -${3*pi/4}" parent="back"/>
   <!-- ros_control plugin -->
   <gazebo>
@@ -21,9 +33,3 @@
     </plugin>
   </gazebo>
-  <!-- first link -->
-  <xacro:body sensors="none"/>
-  <xacro:leg n="0" x="131.56" y="75.45" angle="${1*pi/4}" parent="front"/>
-  <xacro:leg n="1" x="131.56" y="-75.45" angle="-${1*pi/4}" parent="front"/>
-  <xacro:leg n="2" x="-122.56" y="75" angle="${3*pi/4}" parent="back"/>
-  <xacro:leg n="3" x="-122.56" y="-75" angle="-${3*pi/4}" parent="back"/>
 </robot>
