Commit message: update inertia and scale for match true dimensions

File: quaro_description/urdf/body/body.0.0.xacro (robot description, xacro)
@@ -2,4 +2,8 @@
 <robot name="quaro-body" xmlns:xacro="http://ros.org/wiki/xacro">
   <!-- Sensor param will be used later when stereo camera and other sensors will be installed. -->
+  <!-- 0 value in the inertia tensor can cause the robot to crash and
+       sets the link to their origin in the world frame.
+  -->
+  <xacro:property name="zero" value="1"/>
   <xacro:macro name="body" params="sensors">
   <link name="back">
@@ -12,12 +16,12 @@
     </visual>
     <inertial>
-      <mass value="${60*gtoKg}" />
+      <mass value="${125.63*gtoKg}" />
       <origin rpy="0 0 0" xyz="-${54.98*scale} ${0*scale} -${21.33*scale}"/>
-      <inertia  ixx="${1*scale_mm2*gtoKg}"
-                ixy="${0*scale_mm2*gtoKg}"
-                ixz="${0*scale_mm2*gtoKg}"
-                iyy="${1*scale_mm2*gtoKg}"
-                iyz="${0*scale_mm2*gtoKg}"
-                izz="${1*scale_mm2*gtoKg}" />
+      <inertia  ixx="${296016.48*scale_mm2*gtoKg}"
+                ixy="${zero*scale_mm2*gtoKg}"
+                ixz="${148916.20*scale_mm2*gtoKg}"
+                iyy="${593729.76*scale_mm2*gtoKg}"
+                iyz="${zero*scale_mm2*gtoKg}"
+                izz="${691025.98*scale_mm2*gtoKg}" />
     </inertial>
     <collision>
@@ -28,29 +32,5 @@
     </collision>
   </link>
-  <link name="chest-servo">
-    <visual>
-      <geometry>
-        <mesh filename="package://quaro_description/meshes/AX-12A.stl" scale="${scale} ${scale} ${scale}"/>
-      </geometry>
-      <material name="red"/>
-      <origin rpy="0 0 0" xyz="${0*scale} ${0*scale} ${0*scale}"/>
-    </visual>
-    <inertial>
-      <mass value="${60*gtoKg}" />
-      <origin rpy="0 0 0" xyz="${12.61*scale} ${0*scale} ${1.21*scale}"/>
-      <inertia  ixx="${1*scale_mm2*gtoKg}"
-              ixy="${0*scale_mm2*gtoKg}"
-              ixz="${0*scale_mm2*gtoKg}"
-              iyy="${1*scale_mm2*gtoKg}"
-              iyz="${0*scale_mm2*gtoKg}"
-              izz="${1*scale_mm2*gtoKg}" />
-    </inertial>
-    <collision>
-       <geometry>
-         <mesh filename="package://quaro_description/meshes/AX-12A.stl" scale="${scale} ${scale} ${scale}"/>
-       </geometry>
-       <origin rpy="0 0 0" xyz="${0*scale} ${0*scale} ${0*scale}"/>
-     </collision>
-  </link>
+  <xacro:ax12a name="chest-servo" rpy="0 0 0" color="gray"/>
   <link name="spine">
     <visual>
@@ -62,12 +42,12 @@
     </visual>
     <inertial>
-      <mass value="${60*gtoKg}" />
-      <origin rpy="0 0 0" xyz="${0*scale} -${0.56*scale} ${0*scale}"/>
-      <inertia  ixx="${1*scale_mm2*gtoKg}"
-                ixy="${0*scale_mm2*gtoKg}"
-                ixz="${0*scale_mm2*gtoKg}"
-                iyy="${1*scale_mm2*gtoKg}"
-                iyz="${0*scale_mm2*gtoKg}"
-                izz="${1*scale_mm2*gtoKg}" />
+      <mass value="${15.89*gtoKg}" />
+      <origin rpy="0 0 0" xyz="${16.58*scale} -${0.56*scale} ${0*scale}"/>
+      <inertia  ixx="${5271.72*scale_mm2*gtoKg}"
+                ixy="${117.19*scale_mm2*gtoKg}"
+                ixz="${zero*scale_mm2*gtoKg}"
+                iyy="${3500.43*scale_mm2*gtoKg}"
+                iyz="${0.01*scale_mm2*gtoKg}"
+                izz="${5925.70*scale_mm2*gtoKg}" />
     </inertial>
     <collision>
@@ -87,12 +67,12 @@
     </visual>
     <inertial>
-      <mass value="${60*gtoKg}" />
-      <origin rpy="0 0 0" xyz="${71.80*scale} ${0*scale} -${24.62*scale}"/>
-      <inertia  ixx="${1*scale_mm2*gtoKg}"
-                ixy="${0*scale_mm2*gtoKg}"
-                ixz="${0*scale_mm2*gtoKg}"
-                iyy="${1*scale_mm2*gtoKg}"
-                iyz="${0*scale_mm2*gtoKg}"
-                izz="${1*scale_mm2*gtoKg}" />
+      <mass value="${128.96*gtoKg}" />
+      <origin rpy="0 0 0" xyz="${71.80*scale} ${0.05*scale} -${24.62*scale}"/>
+      <inertia  ixx="${327047.38*scale_mm2*gtoKg}"
+                ixy="${314.55*scale_mm2*gtoKg}"
+                ixz="${-219751.03*scale_mm2*gtoKg}"
+                iyy="${984722.31*scale_mm2*gtoKg}"
+                iyz="${-22.94*scale_mm2*gtoKg}"
+                izz="${1072193.50*scale_mm2*gtoKg}" />
     </inertial>
     <collision>
@@ -113,5 +93,5 @@
     <origin rpy="${-pi/2} ${0} ${-pi}" xyz="-${0*scale} -${0*scale} ${0*scale}"/>
     <axis xyz="0 1 0"/>
-    <limit effort="1000.0" lower="${-pi/2}" upper="${pi/2}" velocity="0.5"/>
+    <limit effort="100000.0" lower="${-pi/2}" upper="${pi/2}" velocity="0.5"/>
   </joint>
   <joint name="last" type="fixed">

File: quaro_description/urdf/leg/leg.0.0.xacro (robot description, xacro)
@@ -3,30 +3,10 @@
   <!-- parameter n is the leg number-->
   <xacro:macro name="leg" params="n x y z rpy parent">
+    <!-- 0 value in the inertia tensor can cause the robot to crash and
+         sets the link to their origin in the world frame.
+    -->
+    <xacro:property name="zero" value="1"/>
     <!-- first link -->
-    <link name="hip${n}-servo">
-      <visual>
-        <geometry>
-          <mesh filename="package://quaro_description/meshes/AX-12A.stl" scale="${scale} ${scale} ${scale}"/>
-        </geometry>
-        <material name="red"/>
-        <origin rpy="0 ${pi} 0" xyz="${0*scale} ${0*scale} ${0*scale}"/>
-      </visual>
-      <inertial>
-        <mass value="${60*gtoKg}" />
-        <origin rpy="0 0 0" xyz="${12.61*scale} ${0*scale} ${1.21*scale}"/>
-        <inertia  ixx="${1*scale_mm2*gtoKg}"
-                ixy="${0*scale_mm2*gtoKg}"
-                ixz="${0*scale_mm2*gtoKg}"
-                iyy="${1*scale_mm2*gtoKg}"
-                iyz="${0*scale_mm2*gtoKg}"
-                izz="${1*scale_mm2*gtoKg}" />
-      </inertial>
-      <collision>
-         <geometry>
-           <mesh filename="package://quaro_description/meshes/AX-12A.stl" scale="${scale} ${scale} ${scale}"/>
-         </geometry>
-         <origin rpy="0 ${pi} 0" xyz="${0*scale} ${0*scale} ${0*scale}"/>
-       </collision>
-    </link>
+    <xacro:ax12a name="hip${n}-servo" rpy="0 ${pi} 0" color="red"/>
     <joint name="hip-link${n}" type="fixed">
       <parent link="${parent}"/>
@@ -43,12 +23,12 @@
       </visual>
       <inertial>
-        <mass value="${60*gtoKg}" />
+        <mass value="${19.19*gtoKg}" />
         <origin rpy="${pi} 0 ${pi/2}" xyz="${24.10*scale} -${0*scale} -${0*scale}"/>
-        <inertia  ixx="${1*scale_mm2*gtoKg}"
-                ixy="${0*scale_mm2*gtoKg}"
-                ixz="${0*scale_mm2*gtoKg}"
-                iyy="${1*scale_mm2*gtoKg}"
-                iyz="${0*scale_mm2*gtoKg}"
-                izz="${1*scale_mm2*gtoKg}" />
+        <inertia  ixx="${1783.52*scale_mm2*gtoKg}"
+                ixy="${zero*scale_mm2*gtoKg}"
+                ixz="${zero*scale_mm2*gtoKg}"
+                iyy="${6524.07*scale_mm2*gtoKg}"
+                iyz="${-170.99*scale_mm2*gtoKg}"
+                izz="${6788.11*scale_mm2*gtoKg}" />
       </inertial>
       <collision>
@@ -64,31 +44,7 @@
       <origin rpy="0 0 0" xyz="${0*scale} ${0*scale} ${0*scale}"/>
       <axis xyz="0 0 1"/>
-      <limit effort="1000.0" lower="${-pi/3}" upper="${pi/3}" velocity="0.5"/>
+      <limit effort="100000.0" lower="${-pi/3}" upper="${pi/3}" velocity="0.5"/>
     </joint>
-    <link name="knee${n}-servo">
-      <visual>
-        <geometry>
-          <mesh filename="package://quaro_description/meshes/AX-12A.stl" scale="${scale} ${scale} ${scale}"/>
-        </geometry>
-        <material name="blue"/>
-        <origin rpy="${0} 0 ${0}" xyz="-${0*scale} -${0*scale} ${0*scale}"/>
-      </visual>
-      <inertial>
-        <mass value="${60*gtoKg}" />
-        <origin rpy="0 0 0" xyz="${12.61*scale} ${0*scale} ${1.21*scale}"/>
-        <inertia  ixx="${1*scale_mm2*gtoKg}"
-                ixy="${0*scale_mm2*gtoKg}"
-                ixz="${0*scale_mm2*gtoKg}"
-                iyy="${1*scale_mm2*gtoKg}"
-                iyz="${0*scale_mm2*gtoKg}"
-                izz="${1*scale_mm2*gtoKg}" />
-      </inertial>
-      <collision>
-         <geometry>
-           <mesh filename="package://quaro_description/meshes/AX-12A.stl" scale="${scale} ${scale} ${scale}"/>
-         </geometry>
-         <origin rpy="0 0 0" xyz="${0*scale} ${0*scale} ${0*scale}"/>
-       </collision>
-    </link>
+    <xacro:ax12a name="knee${n}-servo" rpy="0 0 0" color="blue"/>
     <joint name="knee${n}-link" type="fixed">
       <parent link="thigh${n}"/>
@@ -105,12 +61,12 @@
       </visual>
       <inertial>
-        <mass value="${60*gtoKg}" />
+        <mass value="${20.73*gtoKg}" />
         <origin rpy="${0} ${pi/2} ${pi/2}" xyz="-${23.63*scale} ${0*scale} ${0.31*scale}"/>
-        <inertia  ixx="${1*scale_mm2*gtoKg}"
-                ixy="${0*scale_mm2*gtoKg}"
-                ixz="${0*scale_mm2*gtoKg}"
-                iyy="${1*scale_mm2*gtoKg}"
-                iyz="${0*scale_mm2*gtoKg}"
-                izz="${1*scale_mm2*gtoKg}" />
+        <inertia  ixx="${8962.80*scale_mm2*gtoKg}"
+                ixy="${-167.48*scale_mm2*gtoKg}"
+                ixz="${zero*scale_mm2*gtoKg}"
+                iyy="${6916.45*scale_mm2*gtoKg}"
+                iyz="${zero*scale_mm2*gtoKg}"
+                izz="${10135.24*scale_mm2*gtoKg}" />
       </inertial>
       <collision>
@@ -126,31 +82,7 @@
       <origin rpy="0 0 0" xyz="${0*scale} 0 0"/>
       <axis xyz="0 0 1"/>
-      <limit effort="1000.0" lower="${-pi/3}" upper="${pi/3}" velocity="0.5"/>
+      <limit effort="100000.0" lower="${-pi/3}" upper="${pi/3}" velocity="0.5"/>
     </joint>
-    <link name="ankle${n}-servo">
-      <visual>
-        <geometry>
-          <mesh filename="package://quaro_description/meshes/AX-12A.stl" scale="${scale} ${scale} ${scale}"/>
-        </geometry>
-        <material name="green"/>
-        <origin rpy="${0} 0 ${0}" xyz="-${0*scale} -${0*scale} ${0*scale}"/>
-      </visual>
-      <inertial>
-        <mass value="${60*gtoKg}" />
-        <inertia  ixx="${1*scale_mm2*gtoKg}"
-                ixy="${0*scale_mm2*gtoKg}"
-                ixz="${0*scale_mm2*gtoKg}"
-                iyy="${1*scale_mm2*gtoKg}"
-                iyz="${0*scale_mm2*gtoKg}"
-                izz="${1*scale_mm2*gtoKg}" />
-      </inertial>
-      <origin rpy="0 0 0" xyz="${12.61*scale} ${0*scale} ${1.21*scale}"/>
-      <collision>
-         <geometry>
-           <mesh filename="package://quaro_description/meshes/AX-12A.stl" scale="${scale} ${scale} ${scale}"/>
-         </geometry>
-         <origin rpy="0 0 0" xyz="${0*scale} -${0*scale} -${0*scale}"/>
-       </collision>
-    </link>
+    <xacro:ax12a name="ankle${n}-servo" rpy="0 0 0" color="green"/>
     <joint name="ankle${n}-link" type="fixed">
       <parent link="shin${n}"/>
@@ -167,12 +99,12 @@
       </visual>
       <inertial>
-        <mass value="${60*gtoKg}" />
+        <mass value="${27.98*gtoKg}" />
         <origin ryp="0 0 0" xyz="${35.02*scale} -${28.64*scale} ${2.64*scale}"/>
-        <inertia  ixx="${1*scale_mm2*gtoKg}"
-                ixy="${0*scale_mm2*gtoKg}"
-                ixz="${0*scale_mm2*gtoKg}"
-                iyy="${1*scale_mm2*gtoKg}"
-                iyz="${0*scale_mm2*gtoKg}"
-                izz="${1*scale_mm2*gtoKg}" />
+        <inertia  ixx="${44410.23*scale_mm2*gtoKg}"
+                ixy="${-22384.35*scale_mm2*gtoKg}"
+                ixz="${-249.17*scale_mm2*gtoKg}"
+                iyy="${20692.66*scale_mm2*gtoKg}"
+                iyz="${202.94*scale_mm2*gtoKg}"
+                izz="${55471.08*scale_mm2*gtoKg}" />
       </inertial>
       <collision>
@@ -188,5 +120,5 @@
       <origin rpy="0 ${pi} 0" xyz="${0*scale} 0 0"/>
       <axis xyz="0 0 1"/>
-      <limit effort="1000.0" lower="${-pi/3}" upper="${pi/3}" velocity="0.5"/>
+      <limit effort="100000.0" lower="${-pi/3}" upper="${pi/3}" velocity="0.5"/>
     </joint>
   </xacro:macro>

File: quaro_description/urdf/quaro.xacro (robot description, xacro)
@@ -7,6 +7,7 @@
   <xacro:include filename="$(find quaro_description)/urdf/body/body${version}.xacro"/>
   <xacro:include filename="$(find quaro_description)/urdf/quaro.gazebo.xacro"/>
-  <xacro:property name="scale" value="${0.01}"/>
-  <xacro:property name="scale_mm" value="${1e-3*scale}"/>
+  <xacro:include filename="$(find quaro_description)/urdf/common/ax12a.xacro"/>
+  <xacro:property name="scale" value="${1e-3}"/>
+  <xacro:property name="scale_mm" value="${1*scale}"/>
   <xacro:property name="scale_mm2" value="${scale_mm*scale_mm}"/>
   <xacro:property name="gtoKg" value="1e-3"/>
@@ -18,5 +19,5 @@
     <parent link="dummy-link"/>
     <child link="back"/>
-    <origin rpy="0 0 0" xyz="${0*scale} ${0*scale} ${200*scale}"/>
+    <origin rpy="0 0 0" xyz="${0*scale} ${0*scale} ${150*scale}"/>
   </joint>
   <xacro:body sensors="none"/>

Commit message: addapted mesh files to work in gazebo correctly

File: quaro_description/urdf/body/body.0.0.xacro (robot description, xacro)
@@ -5,5 +5,7 @@
        sets the link to their origin in the world frame.
   -->
-  <xacro:property name="zero" value="1"/>
+  <xacro:property name="zero" value="0.1"/>
+  <xacro:property name="effort" value="50"/>
+  <xacro:property name="velocity" value='0.1'/>
   <xacro:macro name="body" params="sensors">
   <link name="back">
@@ -93,5 +95,5 @@
     <origin rpy="${-pi/2} ${0} ${-pi}" xyz="-${0*scale} -${0*scale} ${0*scale}"/>
     <axis xyz="0 1 0"/>
-    <limit effort="100000.0" lower="${-pi/2}" upper="${pi/2}" velocity="0.5"/>
+    <limit effort="${effort}" lower="${-pi/3}" upper="${pi/3}" velocity="${velocity}"/>
   </joint>
   <joint name="last" type="fixed">

File: quaro_description/urdf/leg/leg.0.0.xacro (robot description, xacro)
@@ -6,5 +6,7 @@
          sets the link to their origin in the world frame.
     -->
-    <xacro:property name="zero" value="1"/>
+    <xacro:property name="zero" value="0.0"/>
+    <xacro:property name="effort" value="50"/>
+    <xacro:property name="velocity" value='0.1'/>
     <!-- first link -->
     <xacro:ax12a name="hip${n}-servo" rpy="0 ${pi} 0" color="red"/>
@@ -44,5 +46,5 @@
       <origin rpy="0 0 0" xyz="${0*scale} ${0*scale} ${0*scale}"/>
       <axis xyz="0 0 1"/>
-      <limit effort="100000.0" lower="${-pi/3}" upper="${pi/3}" velocity="0.5"/>
+      <limit effort="${effort}" lower="${-pi/3}" upper="${pi/3}" velocity="${velocity}"/>
     </joint>
     <xacro:ax12a name="knee${n}-servo" rpy="0 0 0" color="blue"/>
@@ -82,5 +84,5 @@
       <origin rpy="0 0 0" xyz="${0*scale} 0 0"/>
       <axis xyz="0 0 1"/>
-      <limit effort="100000.0" lower="${-pi/3}" upper="${pi/3}" velocity="0.5"/>
+      <limit effort="${effort}" lower="${-pi/3}" upper="${pi/3}" velocity="${velocity}"/>
     </joint>
     <xacro:ax12a name="ankle${n}-servo" rpy="0 0 0" color="green"/>
@@ -108,4 +110,12 @@
                 izz="${55471.08*scale_mm2*gtoKg}" />
       </inertial>
+      <surface>
+        <friction>
+          <ode>
+            <mu>1</mu>
+            <mu2>1</mu2>
+          </ode>
+        </friction>
+      </surface>
       <collision>
          <geometry>
@@ -120,5 +130,5 @@
       <origin rpy="0 ${pi} 0" xyz="${0*scale} 0 0"/>
       <axis xyz="0 0 1"/>
-      <limit effort="100000.0" lower="${-pi/3}" upper="${pi/3}" velocity="0.5"/>
+      <limit effort="${effort}" lower="${-pi/3}" upper="${pi/3}" velocity="${velocity}"/>
     </joint>
   </xacro:macro>

File: quaro_description/urdf/quaro.gazebo.xacro (robot description, xacro)
@@ -104,3 +104,11 @@
   <xacro:leg_gazebo n="2"/>
   <xacro:leg_gazebo n="3"/>
+  <!-- ros_control plugin -->
+  <gazebo>
+    <plugin name="gazebo_ros_control" filename="libgazebo_ros_control.so">
+      <robotNamespace>/quaro</robotNamespace>
+      <robotSimType>gazebo_ros_control/DefaultRobotHWSim</robotSimType>
+      <legacyModeNS>true</legacyModeNS>
+    </plugin>
+  </gazebo>
 </robot>

File: quaro_description/urdf/quaro.xacro (robot description, xacro)
@@ -26,11 +26,3 @@
   <xacro:leg n="2" x="-107.63" y="74.77" z="-21" rpy="0 0 ${3*pi/4}" parent="back"/>
   <xacro:leg n="3" x="-107.63" y="-74.77" z="-21" rpy="0 0 -${3*pi/4}" parent="back"/>
-  <!-- ros_control plugin -->
-  <gazebo>
-    <plugin name="gazebo_ros_control" filename="libgazebo_ros_control.so">
-      <robotNamespace>/quaro</robotNamespace>
-      <robotSimType>gazebo_ros_control/DefaultRobotHWSim</robotSimType>
-      <legacyModeNS>true</legacyModeNS>
-    </plugin>
-  </gazebo>
 </robot>

Commit message: ajusted the value for the rpm and effort of the ax12a

File: quaro_description/urdf/body/body.0.0.xacro (robot description, xacro)
@@ -6,6 +6,8 @@
   -->
   <xacro:property name="zero" value="0.1"/>
-  <xacro:property name="effort" value="50"/>
-  <xacro:property name="velocity" value='0.1'/>
+  <!-- Servo does 15kgf.cm-->
+  <xacro:property name="effort" value="1.471"/>
+  <!-- Servo has a rotation of 59 RPM -> 6.178465545 rad/sec -->
+  <xacro:property name="velocity" value='6.178465545'/>
   <xacro:macro name="body" params="sensors">
   <link name="back">

File: quaro_description/urdf/common/ax12a.xacro (robot description, xacro)
@@ -11,5 +11,5 @@
       </visual>
       <inertial>
-        <mass value="${43.01*gtoKg}" />
+        <mass value="${53.01*gtoKg}" />
         <origin rpy="${rpy}" xyz="${12.61*scale} ${0*scale} ${1.21*scale}"/>
         <inertia  ixx="${6917994*scale_mm2*gtoKg}"

File: quaro_description/urdf/leg/leg.0.0.xacro (robot description, xacro)
@@ -7,5 +7,5 @@
     -->
     <xacro:property name="zero" value="0.0"/>
-    <xacro:property name="effort" value="50"/>
+    <xacro:property name="effort" value="1.47"/>
     <xacro:property name="velocity" value='0.1'/>
     <!-- first link -->
