Commit message: add joint state publisher to gazebo launch file. Indented body in body.0.0.xacro. Added todo list

File: quaro_description/urdf/body/body.0.0.xacro (robot description, xacro)
@@ -11,97 +11,97 @@
   <xacro:property name="velocity" value='6.178465545'/>
   <xacro:macro name="body" params="sensors">
-  <link name="back">
-    <visual>
-      <geometry>
-        <mesh filename="package://quaro_description/meshes/back.stl" scale="${scale} ${scale} ${scale}"/>
-      </geometry>
-      <material name="gray"/>
-      <origin rpy="0 0 0" xyz="${0*scale} 0 ${0*scale}"/>
-    </visual>
-    <inertial>
-      <mass value="${125.63*gtoKg}" />
-      <origin rpy="0 0 0" xyz="-${54.98*scale} ${0*scale} -${21.33*scale}"/>
-      <inertia  ixx="${296016.48*scale_mm2*gtoKg}"
-                ixy="${zero*scale_mm2*gtoKg}"
-                ixz="${148916.20*scale_mm2*gtoKg}"
-                iyy="${593729.76*scale_mm2*gtoKg}"
-                iyz="${zero*scale_mm2*gtoKg}"
-                izz="${691025.98*scale_mm2*gtoKg}" />
-    </inertial>
-    <collision>
-       <geometry>
-         <mesh filename="package://quaro_description/meshes/back.stl" scale="${scale} ${scale} ${scale}"/>
-       </geometry>
-       <origin rpy="0 0 0" xyz="${0*scale} 0 ${0*scale}"/>
-    </collision>
-  </link>
-  <xacro:ax12a name="chest-servo" rpy="0 0 0" color="gray"/>
-  <link name="spine">
-    <visual>
-      <geometry>
-        <mesh filename="package://quaro_description/meshes/link-chest.stl" scale="${scale} ${scale} ${scale}"/>
-      </geometry>
-      <material name="yellow"/>
-      <origin rpy="0 0 0" xyz="${16.58*scale} -${0.56*scale} ${0*scale}"/>
-    </visual>
-    <inertial>
-      <mass value="${15.89*gtoKg}" />
-      <origin rpy="0 0 0" xyz="${16.58*scale} -${0.56*scale} ${0*scale}"/>
-      <inertia  ixx="${5271.72*scale_mm2*gtoKg}"
-                ixy="${117.19*scale_mm2*gtoKg}"
-                ixz="${zero*scale_mm2*gtoKg}"
-                iyy="${3500.43*scale_mm2*gtoKg}"
-                iyz="${0.01*scale_mm2*gtoKg}"
-                izz="${5925.70*scale_mm2*gtoKg}" />
-    </inertial>
-    <collision>
-       <geometry>
-         <mesh filename="package://quaro_description/meshes/link-chest.stl" scale="${scale} ${scale} ${scale}"/>
-       </geometry>
-       <origin rpy="0 0 0" xyz="${16.58*scale} -${0.56*scale} ${0*scale}"/>
-     </collision>
-  </link>
-  <link name="front">
-    <visual>
-      <geometry>
-        <mesh filename="package://quaro_description/meshes/front.stl" scale="${scale} ${scale} ${scale}"/>
-      </geometry>
-      <material name="pink"/>
-      <origin rpy="${0} ${0} ${0}" xyz="${0*scale} ${0*scale} ${0*scale}"/>
-    </visual>
-    <inertial>
-      <mass value="${128.96*gtoKg}" />
-      <origin rpy="0 0 0" xyz="${71.80*scale} ${0.05*scale} -${24.62*scale}"/>
-      <inertia  ixx="${327047.38*scale_mm2*gtoKg}"
-                ixy="${314.55*scale_mm2*gtoKg}"
-                ixz="${-219751.03*scale_mm2*gtoKg}"
-                iyy="${984722.31*scale_mm2*gtoKg}"
-                iyz="${-22.94*scale_mm2*gtoKg}"
-                izz="${1072193.50*scale_mm2*gtoKg}" />
-    </inertial>
-    <collision>
-       <geometry>
-         <mesh filename="package://quaro_description/meshes/front.stl" scale="${scale} ${scale} ${scale}"/>
-       </geometry>
-       <origin rpy="0 0 0" xyz="0 0 ${0*scale}"/>
-     </collision>
-  </link>
-  <joint name="servo-link" type="fixed">
-    <parent link="back"/>
-    <child link="chest-servo"/>
-    <origin rpy="${pi/2} ${pi} 0" xyz="${0*scale} -${0.17*scale} -${21*scale}"/>
-  </joint>
-  <joint name="chest" type="revolute">
-    <parent link="chest-servo"/>
-    <child link="spine"/>
-    <origin rpy="${-pi/2} ${0} ${-pi}" xyz="-${0*scale} -${0*scale} ${0*scale}"/>
-    <axis xyz="0 1 0"/>
-    <limit effort="${effort}" lower="${-pi/3}" upper="${pi/3}" velocity="${velocity}"/>
-  </joint>
-  <joint name="last" type="fixed">
-    <parent link="spine"/>
-    <child link="front"/>
-    <origin ryp="${0} ${0} ${0}" xyz="${16.58*scale} ${0*scale} ${21*scale}"/>
-  </joint>
+    <link name="back">
+      <visual>
+        <geometry>
+          <mesh filename="package://quaro_description/meshes/back.stl" scale="${scale} ${scale} ${scale}"/>
+        </geometry>
+        <material name="gray"/>
+        <origin rpy="0 0 0" xyz="${0*scale} 0 ${0*scale}"/>
+      </visual>
+      <inertial>
+        <mass value="${125.63*gtoKg}" />
+        <origin rpy="0 0 0" xyz="-${54.98*scale} ${0*scale} -${21.33*scale}"/>
+        <inertia  ixx="${296016.48*scale_mm2*gtoKg}"
+                  ixy="${zero*scale_mm2*gtoKg}"
+                  ixz="${148916.20*scale_mm2*gtoKg}"
+                  iyy="${593729.76*scale_mm2*gtoKg}"
+                  iyz="${zero*scale_mm2*gtoKg}"
+                  izz="${691025.98*scale_mm2*gtoKg}" />
+      </inertial>
+      <collision>
+        <geometry>
+          <mesh filename="package://quaro_description/meshes/back.stl" scale="${scale} ${scale} ${scale}"/>
+        </geometry>
+        <origin rpy="0 0 0" xyz="${0*scale} 0 ${0*scale}"/>
+      </collision>
+    </link>
+    <xacro:ax12a name="chest-servo" rpy="0 0 0" color="gray"/>
+    <link name="spine">
+      <visual>
+        <geometry>
+          <mesh filename="package://quaro_description/meshes/link-chest.stl" scale="${scale} ${scale} ${scale}"/>
+        </geometry>
+        <material name="yellow"/>
+        <origin rpy="0 0 0" xyz="${16.58*scale} -${0.56*scale} ${0*scale}"/>
+      </visual>
+      <inertial>
+        <mass value="${15.89*gtoKg}" />
+        <origin rpy="0 0 0" xyz="${16.58*scale} -${0.56*scale} ${0*scale}"/>
+        <inertia  ixx="${5271.72*scale_mm2*gtoKg}"
+                  ixy="${117.19*scale_mm2*gtoKg}"
+                  ixz="${zero*scale_mm2*gtoKg}"
+                  iyy="${3500.43*scale_mm2*gtoKg}"
+                  iyz="${0.01*scale_mm2*gtoKg}"
+                  izz="${5925.70*scale_mm2*gtoKg}" />
+      </inertial>
+      <collision>
+        <geometry>
+          <mesh filename="package://quaro_description/meshes/link-chest.stl" scale="${scale} ${scale} ${scale}"/>
+        </geometry>
+        <origin rpy="0 0 0" xyz="${16.58*scale} -${0.56*scale} ${0*scale}"/>
+      </collision>
+    </link>
+    <link name="front">
+      <visual>
+        <geometry>
+          <mesh filename="package://quaro_description/meshes/front.stl" scale="${scale} ${scale} ${scale}"/>
+        </geometry>
+        <material name="pink"/>
+        <origin rpy="${0} ${0} ${0}" xyz="${0*scale} ${0*scale} ${0*scale}"/>
+      </visual>
+      <inertial>
+        <mass value="${128.96*gtoKg}" />
+        <origin rpy="0 0 0" xyz="${71.80*scale} ${0.05*scale} -${24.62*scale}"/>
+        <inertia  ixx="${327047.38*scale_mm2*gtoKg}"
+                  ixy="${314.55*scale_mm2*gtoKg}"
+                  ixz="${-219751.03*scale_mm2*gtoKg}"
+                  iyy="${984722.31*scale_mm2*gtoKg}"
+                  iyz="${-22.94*scale_mm2*gtoKg}"
+                  izz="${1072193.50*scale_mm2*gtoKg}" />
+      </inertial>
+      <collision>
+        <geometry>
+          <mesh filename="package://quaro_description/meshes/front.stl" scale="${scale} ${scale} ${scale}"/>
+        </geometry>
+        <origin rpy="0 0 0" xyz="0 0 ${0*scale}"/>
+      </collision>
+    </link>
+    <joint name="servo-link" type="fixed">
+      <parent link="back"/>
+      <child link="chest-servo"/>
+      <origin rpy="${pi/2} ${pi} 0" xyz="${0*scale} -${0.17*scale} -${21*scale}"/>
+    </joint>
+    <joint name="chest" type="revolute">
+      <parent link="chest-servo"/>
+      <child link="spine"/>
+      <origin rpy="${-pi/2} ${0} ${-pi}" xyz="-${0*scale} -${0*scale} ${0*scale}"/>
+      <axis xyz="0 1 0"/>
+      <limit effort="${effort}" lower="${-pi/3}" upper="${pi/3}" velocity="${velocity}"/>
+    </joint>
+    <joint name="last" type="fixed">
+      <parent link="spine"/>
+      <child link="front"/>
+      <origin ryp="${0} ${0} ${0}" xyz="${16.58*scale} ${0*scale} ${21*scale}"/>
+    </joint>
   </xacro:macro>
 </robot>
